File: hardware/hardware.kicad_sch (KiCad schematic)
At the start: 36 parts, among them SW1 SW_Push_45deg, SW10 SW_Push_45deg, SW11 SW_Push_45deg, SW12 SW_Push_45deg, SW13 SW_Push_45deg, SW14 SW_Push_45deg, SW15 SW_Push_45deg, SW16 SW_Push_45deg, SW17 SW_Push_45deg, SW18 SW_Push_45deg, SW19 SW_Push_45deg, SW2 SW_Push_45deg, SW20 SW_Push_45deg, SW21 SW_Push_45deg, SW22 SW_Push_45deg, SW23 SW_Push_45deg, SW24 SW_Push_45deg, SW25 SW_Push_45deg, SW26 SW_Push_45deg, SW27 SW_Push_45deg, SW28 SW_Push_45deg, SW29 SW_Push_45deg, SW3 SW_Push_45deg, SW30 SW_Push_45deg, SW31 SW_Push_45deg, SW32 SW_Push_45deg, SW33 SW_Push_45deg, SW34 SW_Push_45deg, SW35 SW_Push_45deg, SW36 SW_Push_45deg, SW4 SW_Push_45deg, SW5 SW_Push_45deg, SW6 SW_Push_45deg, SW7 SW_Push_45deg, SW8 SW_Push_45deg, SW9 SW_Push_45deg

Commit message: journalmaxxing
Parts:
- added C1, C13, C14, C16, C2: 1uF/25V, symbol Device:C
- added C10: 10uf/25V, symbol Device:C
- added C11, C3, C4, C5, C6, C7, C9: 1uf/25V, symbol Device:C
- added C12, C15: 4.7uF/25V, symbol Device:C
- added C17, C18: 4.7uF, symbol Device:C
- added C8: 1.8uf/25V, symbol Device:C
- added D1, D2, D3: MBR0530, Diode_SMD:D_SOD-123, symbol Diode:MBR0530
- added J1: 6871XX149022_687126149022, 6871XX149022_687126149022:687126149022, symbol 6871XX149022_687126149022:6871XX149022_687126149022
- added L1: 10uH, symbol Device:L
- added Q1: BSS138, Package_TO_SOT_SMD:SOT-23, symbol Transistor_FET:BSS138
- added R1: 1M, symbol Device:R
- added R2: 0.2, symbol Device:R
- added R3: 5M, symbol Device:R
- added U1: STM32U5A5RJTx, Package_QFP:LQFP-64_10x10mm_P0.5mm, symbol MCU_ST_STM32U5:STM32U5A5RJTx
- added U2: TXB0108PWR, TXB0108PWR:SOP65P640X120-20N, symbol TXB0108PWR:TXB0108PWR
Connections:
- new net: C8.1, J1.26
- new net: C10.1, C9.1, J1.14, J1.15, L1.1
- new net: C12.1, D1.2 (A), L1.2, Q1.3 (D)
- new net: C13.1, C14.1, D1.1 (K), J1.23
- new net: C17.2, U2.2 (VCCA)
- new net: C4.1, J1.18
- new net: C18.2, U2.19 (VCCB)
- new net: C12.2, D2.2 (A), D3.1 (K)
- new net: C15.1, C16.1, D3.2 (A), J1.25
- new net: U1.18 (VSS), U1.31 (VSS), U1.47 (VSS), U1.63 (VSS)
- new net: J1.2, Q1.1 (G), R1.1
- new net: C2.1, J1.4
- new net: C7.1, J1.24
- new net: C1.1, J1.3
- new net: J1.1, Q1.2 (S), R2.2
- new net: C11.1, J1.19
- new net: C6.1, J1.22
- new net: C3.1, J1.17
- new net: C5.1, J1.21
- new net BS0: J1.7
- new net EPD BUSY: U2.13 (B7)
- new net EPD BUSY': J1.8, U2.8 (A7)
- new net EPD CS: U2.15 (B5), U2.16 (B4)
- new net EPD CS': J1.11, U2.5 (A4)
- new net EPD DC': J1.10, U2.6 (A5)
- new net EPD DIN: U2.18 (B2)
- new net EPD DIN': J1.13, U2.3 (A2)
- new net EPD RST: U2.14 (B6)
- new net EPD RST': J1.9, U2.7 (A6)
- new net EPD SCK: U2.17 (B3)
- new net EPD SCK': J1.12, U2.4 (A3)
- new net GND: C1.2, C10.2, C11.2, C13.2, C14.2, C15.2, C16.2, C17.1, C18.1, C2.2, C3.2, C4.2, C5.2, C6.2, C7.2, C8.2, C9.2, D2.1 (K), J1.16, J1.Z1, J1.Z2, R1.2, R2.1, R3.2
Other:
- moved on the sheet: SW1, SW10, SW11, SW12, SW13, SW14, SW15, SW16, SW17, SW18, SW19, SW2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

Commit message: jounal for yesterday's work
Parts:
- added C19: 104?, Capacitor_SMD:C_0805_2012Metric, symbol Device:C
- added C20: 22nF, Capacitor_SMD:C_0805_2012Metric, symbol Device:C
- added C21: 1uF, Capacitor_SMD:C_0805_2012Metric, symbol Device:C
- added C22: 104, Capacitor_SMD:C_0805_2012Metric, symbol Device:C
- added Q2: AO3401A, Package_TO_SOT_SMD:SOT-23, symbol Transistor_FET:AO3401A
- added Q3: S8050, Package_TO_SOT_THT:TO-92_Inline, symbol Transistor_BJT:S8050
- added R10: R, Resistor_SMD:R_1206_3216Metric, symbol Device:R
- added R11, R12, R13, R14, R15, R16, R17, R18: 100, Capacitor_SMD:C_0805_2012Metric, symbol Device:R
- added R4: 100K, Resistor_SMD:R_1206_3216Metric, symbol Device:R
- added R5, R7, R8: 47K, Resistor_SMD:R_1206_3216Metric, symbol Device:R
- added R6: 10K, Resistor_SMD:R_1206_3216Metric, symbol Device:R
- added R9: 1K, Resistor_SMD:R_1206_3216Metric, symbol Device:R
- added SW37: root, footprints:SW_D2LS-11_2_OMR, symbol Switch:SW_Push_45deg
- added U3: RT9193-33GB, RT9193_33GB:SOT94P279X129-5N, symbol RT9193-33GB:RT9193-33GB
- C1, C11, C13, C14, C16, C2, C3, C4, C5, C6, C7, C9: footprint (none) -> Capacitor_SMD:C_0805_2012Metric
- C10, C12, C15, C17, C18, C8: footprint (none) -> Capacitor_SMD:C_1206_3216Metric
- J1: footprint 6871XX149022_687126149022:687126149022 -> 687126149022:687126149022
- L1: footprint (none) -> Inductor_SMD:L_Sunlord_SWPA3012S
- R1, R2, R3: footprint (none) -> Resistor_SMD:R_1206_3216Metric
- SW1: value SW_Push_45deg -> 7; footprint (none) -> footprints:SW_D2LS-11_2_OMR
- SW10: value SW_Push_45deg -> divide_sign; footprint (none) -> footprints:SW_D2LS-11_2_OMR
- SW11: value SW_Push_45deg -> 1; footprint (none) -> footprints:SW_D2LS-11_2_OMR
- SW12: value SW_Push_45deg -> 0; footprint (none) -> footprints:SW_D2LS-11_2_OMR
- SW13: value SW_Push_45deg -> 2; footprint (none) -> footprints:SW_D2LS-11_2_OMR
- SW14: value SW_Push_45deg -> dot; footprint (none) -> footprints:SW_D2LS-11_2_OMR
- SW15: value SW_Push_45deg -> 3; footprint (none) -> footprints:SW_D2LS-11_2_OMR
- SW16: value SW_Push_45deg -> pi; footprint (none) -> footprints:SW_D2LS-11_2_OMR
- SW17: value SW_Push_45deg -> plus_sign; footprint (none) -> footprints:SW_D2LS-11_2_OMR
- SW18: value SW_Push_45deg -> ans; footprint (none) -> footprints:SW_D2LS-11_2_OMR
- SW19: value SW_Push_45deg -> minus_sign; footprint (none) -> footprints:SW_D2LS-11_2_OMR
- SW2: value SW_Push_45deg -> 8; footprint (none) -> footprints:SW_D2LS-11_2_OMR
- SW20: value SW_Push_45deg -> equal_sign; footprint (none) -> footprints:SW_D2LS-11_2_OMR
- SW21: value SW_Push_45deg -> mod; footprint (none) -> footprints:SW_D2LS-11_2_OMR
- SW22: value SW_Push_45deg -> up_arrow; footprint (none) -> footprints:SW_D2LS-11_2_OMR
- SW23: value SW_Push_45deg -> shift; footprint (none) -> footprints:SW_D2LS-11_2_OMR
- SW24: value SW_Push_45deg -> on_button; footprint (none) -> footprints:SW_D2LS-11_2_OMR
- SW25: value SW_Push_45deg -> sin; footprint (none) -> footprints:SW_D2LS-11_2_OMR
- SW26: value SW_Push_45deg -> left_arrow; footprint (none) -> footprints:SW_D2LS-11_2_OMR
- SW27: value SW_Push_45deg -> right_arrow; footprint (none) -> footprints:SW_D2LS-11_2_OMR
- SW28: value SW_Push_45deg -> log; footprint (none) -> footprints:SW_D2LS-11_2_OMR
- SW29: value SW_Push_45deg -> cos; footprint (none) -> footprints:SW_D2LS-11_2_OMR
- SW3: value SW_Push_45deg -> 9; footprint (none) -> footprints:SW_D2LS-11_2_OMR
- SW30: value SW_Push_45deg -> tan; footprint (none) -> footprints:SW_D2LS-11_2_OMR
- SW31: value SW_Push_45deg -> down_arrow; footprint (none) -> footprints:SW_D2LS-11_2_OMR
- SW32: value SW_Push_45deg -> open_parenthesis; footprint (none) -> footprints:SW_D2LS-11_2_OMR
- SW33: value SW_Push_45deg -> todo; footprint (none) -> footprints:SW_D2LS-11_2_OMR
- SW34: value SW_Push_45deg -> closed_parenthesis; footprint (none) -> footprints:SW_D2LS-11_2_OMR
- SW35: value SW_Push_45deg -> ln; footprint (none) -> footprints:SW_D2LS-11_2_OMR
- SW36: value SW_Push_45deg -> elevate; footprint (none) -> footprints:SW_D2LS-11_2_OMR
- SW4: value SW_Push_45deg -> delete; footprint (none) -> footprints:SW_D2LS-11_2_OMR
- SW5: value SW_Push_45deg -> clear; footprint (none) -> footprints:SW_D2LS-11_2_OMR
- SW6: value SW_Push_45deg -> 4; footprint (none) -> footprints:SW_D2LS-11_2_OMR
- SW7: value SW_Push_45deg -> 5; footprint (none) -> footprints:SW_D2LS-11_2_OMR
- SW8: value SW_Push_45deg -> 6; footprint (none) -> footprints:SW_D2LS-11_2_OMR
- SW9: value SW_Push_45deg -> multiply_sign; footprint (none) -> footprints:SW_D2LS-11_2_OMR
Connections:
- net BS0: now also R10.2
- net EPD BUSY: now also U1.4 (PC15)
- net EPD CS: now also U1.20 (PA4)
- net EPD DIN: now also U1.23 (PA7)
- net EPD RST: now also U1.3 (PC14), R6.1, R9.1
- net EPD SCK: now also U1.15 (PA1)
- net GND: now also U2.11 (GND), C19.1, C20.2, C21.1, C22.2, Q3.1 (E), R4.2, R7.2, R8.2, U3.2 (GND)
- net COL 4: now reaches SW17.1, SW18.1, SW24.1, SW28.1, SW35.1, SW36.1, SW4.1, SW9.1
- net COL 4: now also U1.25 (PC5)
- net at SW12.2, SW14.2, SW16.2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: now also R18.1
- net COL 2: now reaches SW13.1, SW14.1, SW2.1, SW22.1, SW26.1, SW31.1, SW32.1, SW7.1
- net COL 2: now also U1.21 (PA5)
- net at SW10.2, SW6.2, SW7.2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: now also R16.1
- net 3V3_OUT: now reaches C17.2, U2.2 (VCCA)
- net 3V3_OUT: now also C21.2, R10.1, U3.5 (VOUT)
- net at SW21.2, SW22.2, SW23.2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: now also R11.1
- net VCC: now reaches C18.2, U2.19 (VCCB)
- net VCC: now also C19.2, Q2.2 (S), U3.1 (VIN)
- net COL 1: now reaches SW1.1, SW11.1, SW12.1, SW21.1, SW25.1, SW29.1, SW30.1, SW6.1
- net COL 1: now also U1.17 (PA3)
- net at SW1.2, SW2.2, SW3.2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: now also R15.1
- net COL 3: now reaches SW15.1, SW16.1, SW23.1, SW27.1, SW3.1, SW33.1, SW34.1, SW8.1
- net COL 3: now also U1.24 (PC4)
- net at SW29.2, SW31.2, SW33.2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: now also R13.1
- net at SW25.2, SW26.2, SW27.2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: now also R12.1
- net ROW 5: now reaches U1.10 (PC2)
- net ROW 5: now also R15.2
- net ROW 6: now reaches U1.11 (PC3)
- net ROW 6: now also R16.2
- net ROW 7: now reaches U1.14 (PA0)
- net ROW 7: now also R17.2
- net ROW 8: now reaches U1.16 (PA2)
- net ROW 8: now also R18.2
- net EPD DC: now reaches U1.2 (PC13)
- net COL 5: now reaches U1.26 (PB0)
- net COL 5: now also SW10.1, SW19.1, SW20.1, SW5.1, SW37.1
- net ROW 1: now reaches U1.5 (PH0)
- net ROW 1: now also R11.2
- net ROW 2: now reaches U1.6 (PH1)
- net ROW 2: now also R12.2
- net ROW 3: now reaches U1.8 (PC0)
- net ROW 3: now also R13.2
- net ROW 4: now reaches U1.9 (PC1)
- net ROW 4: now also R14.2
- net at SW11.2, SW13.2, SW15.2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: now also R17.1
- net at SW30.2, SW32.2, SW34.2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: now also R14.1, SW37.2
- new net: Q2.1 (G), Q3.3 (C), R5.2
- new net: C20.1, U3.4 (BP)
- new net: Q3.2 (B), R6.2, R7.1
- new net VCC EN: R4.1, R8.1, R9.2, U3.3 (EN)
- new net VCC_INT: C22.1, Q2.3 (D), R5.1
Other:
- note added: "This is used to enable 4-line spi"
- moved on the sheet: C1, C10, C11, C12, C13, C14, C15, C16, C2, C3, C4, C5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
